File: GreengrassEntryHardware.kicad_pcb (KiCad board)
At the start: 2 copper layers, 80 x 77 mm, 37 parts, among them J1 USB_B_Micro, J2 GPIOBreakout, J3 Raspberry_Pi_2_3, J4 AutomaticSlidingDoor, J5 MFRC-522, J6 DoorEnable, J8 FEEDBACK, U1 CH340G, Y1 12MHZ

Commit message: Push 5v to the relays
Connections:
- J3 pad 2: (no net) -> Net-(J3-Pad2)
- J4 pad 8: GNDD -> Net-(J3-Pad2)
Routing:
- net Net-(J3-Pad2): track 0.00 -> 85.2 mm, vias 0 -> 2
- net Net-(C1-Pad1): track 55.2 -> 53.8 mm
Changed lines of the file:
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@@
     (thickness 1.6)
     (drawings 24)
-    (tracks 268)
+    (tracks 281)
     (zones 0)
     (modules 37)
-    (nets 51)
+    (nets 52)
   )
   (page A4)
@@
   (net 49 "Net-(J8-Pad2)")
   (net 50 "Net-(J8-Pad3)")
+  (net 51 "Net-(J3-Pad2)")
   (net_class Default "This is the default net class."
     (clearance 0.2)
@@
     (add_net "Net-(J3-Pad10)")
     (add_net "Net-(J3-Pad17)")
+    (add_net "Net-(J3-Pad2)")
     (add_net "Net-(J3-Pad32)")
     (add_net "Net-(J3-Pad8)")
@@
     (fp_line (start 20 -2) (end 20 7) (layer F.SilkS) (width 0.15))
     (pad 8 thru_hole circle (at 17.5 0) (size 2 2) (drill 1) (layers *.Cu *.Mask)
-      (net 9 GNDD))
+      (net 51 "Net-(J3-Pad2)"))
     (pad 7 thru_hole circle (at 15 0) (size 2 2) (drill 1) (layers *.Cu *.Mask)
       (net 33 "Net-(J4-Pad7)"))
@@
     (pad 4 thru_hole oval (at -2.54 2.54 270) (size 1.7 1.7) (drill 1) (layers *.Cu *.Mask))
     (pad 3 thru_hole oval (at 0 2.54 270) (size 1.7 1.7) (drill 1) (layers *.Cu *.Mask))
-    (pad 2 thru_hole oval (at -2.54 0 270) (size 1.7 1.7) (drill 1) (layers *.Cu *.Mask))
+    (pad 2 thru_hole oval (at -2.54 0 270) (size 1.7 1.7) (drill 1) (layers *.Cu *.Mask)
+      (net 51 "Net-(J3-Pad2)"))
     (pad 1 thru_hole rect (at 0 0 270) (size 1.7 1.7) (drill 1) (layers *.Cu *.Mask)
       (net 1 "Net-(C1-Pad1)"))
@@
   (segment (start 163.67142 84.27858) (end 167.5 80.45) (width 0.25) (layer F.Cu) (net 1))
   (segment (start 163.67142 84.32142) (end 163.67142 84.27858) (width 0.25) (layer F.Cu) (net 1))
-  (segment (start 167.5 80.45) (end 167.5 64.3) (width 0.25) (layer B.Cu) (net 1))
-  (segment (start 167.5 64.3) (end 168.875 62.925) (width 0.25) (layer B.Cu) (net 1))
-  (segment (start 172.86 61.24) (end 172.86 60.14) (width 0.25) (layer B.Cu) (net 1))
-  (segment (start 171.175 62.925) (end 172.86 61.24) (width 0.25) (layer B.Cu) (net 1))
-  (segment (start 168.875 62.925) (end 171.175 62.925) (width 0.25) (layer B.Cu) (net 1))
+  (segment (start 172.86 61.24) (end 167.5 66.6) (width 0.25) (layer B.Cu) (net 1))
+  (segment (start 167.5 66.6) (end 167.5 80.45) (width 0.25) (layer B.Cu) (net 1))
+  (segment (start 172.86 60.14) (end 172.86 61.24) (width 0.25) (layer B.Cu) (net 1))
   (segment (start 171.3 91.925) (end 171.3 90.85) (width 0.25) (layer F.Cu) (net 2))
   (segment (start 177.3 101.55) (end 177.3 95.6) (width 0.25) (layer F.Cu) (net 2))
@@
   (segment (start 150.7 124.4) (end 150.8 124.5) (width 0.25) (layer B.Cu) (net 50))
   (segment (start 150.7 117) (end 150.7 124.4) (width 0.25) (layer B.Cu) (net 50))
+  (via (at 167.8 64.3) (size 1.2) (drill 0.9) (layers F.Cu B.Cu) (net 51))
+  (segment (start 171.495001 60.704001) (end 167.899002 64.3) (width 0.25) (layer B.Cu) (net 51))
+  (segment (start 171.495001 58.964999) (end 171.495001 60.704001) (width 0.25) (layer B.Cu) (net 51))
+  (segment (start 167.899002 64.3) (end 167.8 64.3) (width 0.25) (layer B.Cu) (net 51))
+  (segment (start 172.86 57.6) (end 171.495001 58.964999) (width 0.25) (layer B.Cu) (net 51))
+  (segment (start 167.8 64.3) (end 163.3 68.8) (width 0.25) (layer F.Cu) (net 51))
+  (segment (start 163.3 68.8) (end 163.3 74.3) (width 0.25) (layer F.Cu) (net 51))
+  (segment (start 147 90.6) (end 147 107.1) (width 0.25) (layer F.Cu) (net 51))
+  (segment (start 163.3 74.3) (end 147 90.6) (width 0.25) (layer F.Cu) (net 51))
+  (segment (start 147 107.1) (end 143.6 110.5) (width 0.25) (layer F.Cu) (net 51))
+  (via (at 133.3 120.8) (size 1.2) (drill 0.9) (layers F.Cu B.Cu) (net 51))
+  (segment (start 143.6 110.5) (end 133.3 120.8) (width 0.25) (layer F.Cu) (net 51))
+  (segment (start 133.3 120.8) (end 131.9 120.8) (width 0.25) (layer B.Cu) (net 51))
+  (segment (start 130.7 122) (end 130.7 124.5) (width 0.25) (layer B.Cu) (net 51))
+  (segment (start 131.9 120.8) (end 130.7 122) (width 0.25) (layer B.Cu) (net 51))
   (zone (net 9) (net_name GNDD) (layer F.Cu) (hatch edge 0.508)
     (connect_pads (clearance 0.508))
     (min_thickness 0.254)
-    (fill (arc_segments 32) (thermal_gap 0.508) (thermal_bridge_width 0.508))
+    (fill yes (arc_segments 32) (thermal_gap 0.508) (thermal_bridge_width 0.508))
     (polygon
       (pts
@@
     (connect_pads (clearance 0.508))
     (min_thickness 0.254)
-    (fill (arc_segments 32) (thermal_gap 0.508) (thermal_bridge_width 0.508))
+    (fill yes (arc_segments 32) (thermal_gap 0.508) (thermal_bridge_width 0.508))
     (polygon
       (pts
